Commit message: Update 1811
Analytical Cartesian Planner
Updates URDF for IAAC setup

File: data/robots/ur10e.urdf (robot description, URDF)
Before this commit: robot ur10e_robot, 11 links, 10 joints
Joints:
- joint base_link-base_link_inertia: origin xyz=0 0 0 rpy=0 0 3.141592653589793 -> xyz=0 0 0 rpy=0 0 -3.14
- joint shoulder_lift_joint: limit lower=-6.283185307179586 upper=6.283185307179586 effort=330.0 velocity=2.0943951023931953 -> lower=-3.14 upper=0 effort=330.0 velocity=2.0943951023931953
- joint shoulder_pan_joint: limit lower=-6.283185307179586 upper=6.283185307179586 effort=330.0 velocity=2.0943951023931953 -> lower=-6.2831 upper=6.2831 effort=330.0 velocity=2.0943951023931953
